File: squid_board/Kamioka_SQUID_board_v1.kicad_sch (KiCad schematic)
At the start: 18 parts, among them J1 Conn_01x25, J6 Conn_01x51

Commit message: add SQUID board changes
Parts:
- SQ1, SQ2, SQ3, SQ4: value ~ -> (none)

Commit message: Clean up ground paths and add new stepfile
Connections:
- net GND: now also SQ1.10 (th2), SQ1.11, SQ1.3 (th1), SQ1.5 (H-), SQ2.10 (th2), SQ2.11, SQ2.3 (th1), SQ2.5 (H-), SQ3.10 (th2), SQ3.11, SQ3.3 (th1), SQ3.5 (H-), SQ4.10 (th2), SQ4.11, SQ4.3 (th1), SQ4.5 (H-); no longer SQ1.4 (H-), SQ1.9, SQ2.4 (H-), SQ2.9, SQ3.4 (H-), SQ3.9, SQ4.4 (H-), SQ4.9
- net I+_sq1: now also SQ1.8 (Vsq-); no longer SQ1.7 (Vsq-)
- net I+sq_2: now also SQ2.8 (Vsq-); no longer SQ2.7 (Vsq-)
- net I+sq_3: now also SQ3.8 (Vsq-); no longer SQ3.7 (Vsq-)
- net I+sq_4: now also SQ4.8 (Vsq-); no longer SQ4.7 (Vsq-)
- net I-sq_1: now also SQ1.9 (Vsq+); no longer SQ1.8 (Vsq+)
- net I-sq_2: now also SQ2.9 (Vsq+); no longer SQ2.8 (Vsq+)
- net I-sq_3: now also SQ3.9 (Vsq+); no longer SQ3.8 (Vsq+)
- net I-sq_4: now also SQ4.9 (Vsq+); no longer SQ4.8 (Vsq+)
- net fb+sq_1: now also SQ1.6 (fb+); no longer SQ1.5 (fb+)
- net fb+sq_2: now also SQ2.6 (fb+); no longer SQ2.5 (fb+)
- net fb+sq_3: now also SQ3.6 (fb+); no longer SQ3.5 (fb+)
- net fb+sq_4: now also SQ4.6 (fb+); no longer SQ4.5 (fb+)
- net fb-sq_1: now also SQ1.7 (fb-); no longer SQ1.6 (fb-)
- net fb-sq_2: now also SQ2.7 (fb-); no longer SQ2.6 (fb-)
- net fb-sq_3: now also SQ3.7 (fb-); no longer SQ3.6 (fb-)
- net fb-sq_4: now also SQ4.7 (fb-); no longer SQ4.6 (fb-)
- net h+sq_1: now also SQ1.4 (H+); no longer SQ1.3 (H+)
- net h+sq_2: now also SQ2.4 (H+); no longer SQ2.3 (H+)
- net h+sq_3: now also SQ3.4 (H+); no longer SQ3.3 (H+)
- net h+sq_4: now also SQ4.4 (H+); no longer SQ4.3 (H+)

Commit message: latest update
Parts:
- added H10, H11, H12, H13, H14, H15, H16, H17, H18, H19, H20, H9: MountingHole_Pad, MountingHole:MountingHole_2.2mm_M2_DIN965_Pad_TopBottom, symbol Mechanical:MountingHole_Pad
- J1: footprint (none) -> coldMount_footprints_src:MDM25-SBSP; symbol Connector_Generic:Conn_01x25 -> Connector_Generic:Conn_01x27
- J6: symbol Connector_Generic:Conn_01x51 -> Connector_Generic:Conn_01x53
Connections:
- net GND: now also J1.MH1 (Pin_26), J1.MH2 (Pin_27), J6.MH1 (Pin_52), J6.MH2 (Pin_53), H10.1, H11.1, H12.1, H13.1, H14.1, H15.1, H16.1, H17.1, H18.1, H19.1, H20.1, H9.1

Commit message: add udpated pcb
Parts:
- added C1, C2, C3, C4, C5, C6, C7, C8: C, Capacitor_SMD:C_0805_2012Metric, symbol Device:C
- added R10, R11, R12, R13, R14, R15, R16, R9: R_US, Capacitor_SMD:C_0805_2012Metric, symbol Device:R_US
- added R5, R6, R7, R8: R_US, Resistor_SMD:R_0805_2012Metric, symbol Device:R_US
Connections:
- net Ch1_3: now also R5.2
- net Ch2_3: now also R6.2
- net Ch3_3: now also R7.2
- net Ch4_3: now also R8.2
- net I+_sq1: now also C5.1, R9.2
- net I+sq_2: now also C6.1, R10.2
- net I+sq_3: now also C7.1, R11.2
- net I+sq_4: now also C8.1, R12.2
- net I-sq_1: now also C5.2, R9.1
- net I-sq_2: now also C6.2, R10.1
- net I-sq_3: now also C7.2, R11.1
- net I-sq_4: now also C8.2, R12.1
- net b+TES1: now also C1.2
- net b+TES2: now also C2.2
- net b+TES3: now also C3.2
- net b+TES4: now also C4.2
- net fb+sq_1: now also R13.1
- net fb+sq_2: now also R14.1
- net fb+sq_3: now also R15.1
- net fb+sq_4: now also R16.1
- net fb-sq_1: now also R13.2
- net fb-sq_2: now also R14.2
- net fb-sq_3: now also R15.2
- net fb-sq_4: now also R16.2
- new net: C1.1, R5.1
- new net: C2.1, R6.1
- new net: C3.1, R7.1
- new net: C4.1, R8.1
